File: main_indoor_sensor.brd (EAGLE design)
At the start: 12 parts

Commit message: Version 0.1 avec prototype créé
Parts:
- added R5: (no value), eagle-ltspice:0204/7
- moved U$2 6.35 mm to (92.7, 48.3)
- moved U$5 5.08 mm to (64.8, 41.9)
- moved U$8 3.42 mm to (71.1, 46.4)
- moved R3 1.27 mm to (36.8, 61.0)
Connections:
- new net N$19: R5.1, U$7.VCC
- net RASTNEST: now also R5.2; no longer U$7.VCC
Routing:
- net N$4: track 15.2 -> 40.6 mm
- net N$3: track 30.5 -> 50.8 mm
- net GND: track 0.00 -> 14.0 mm, vias 0 -> 2
- net RASTNEST: track 120.7 -> 109.2 mm, vias 0 -> 2
- net N$1: track 8.89 -> 20.3 mm
- net N$19: track 0.00 -> 8.43 mm
- net N$7: track 43.2 -> 48.3 mm, vias 0 -> 2
- net N$10: track 3.81 -> 6.35 mm
- net N$2: track 14.0 -> 15.2 mm
- net N$12: track 16.5 -> 17.8 mm
- net N$8: vias 2 -> 0
- net N$15: vias 1 -> 0
