File: main_indoor_sensor.sch (EAGLE design)
At the start: 12 parts

Commit message: Version 0.1 avec prototype créé
Parts:
- added R5: (no value), eagle-ltspice:R0204/7
Connections:
- new net N$19: R5.1, U$7.VV
- net RASTNEST: now also R5.2; no longer U$7.VV
Changed lines of the file:
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@@
 <part name="R4" library="eagle-ltspice" deviceset="R" device="0204/7"/>
 <part name="U$7" library="piweather" deviceset="KRS0612" device="PUSH"/>
-<part name="P+7" library="supply1" deviceset="VCC" device=""/>
 <part name="GND9" library="supply1" deviceset="GND" device=""/>
 <part name="U$8" library="piweather" deviceset="NCP1402" device="SPARKFUN"/>
 <part name="GND10" library="supply1" deviceset="GND" device=""/>
 <part name="P+6" library="supply1" deviceset="VCC" device=""/>
+<part name="R5" library="eagle-ltspice" deviceset="R" device="0204/7"/>
 </parts>
 <sheets>
@@
 <instance part="R4" gate="G$1" x="-50.8" y="-25.4"/>
 <instance part="U$7" gate="G$1" x="-33.02" y="43.18"/>
-<instance part="P+7" gate="VCC" x="-50.8" y="50.8"/>
 <instance part="GND9" gate="1" x="-50.8" y="30.48"/>
 <instance part="U$8" gate="G$1" x="0" y="48.26"/>
 <instance part="GND10" gate="1" x="-10.16" y="66.04" rot="R180"/>
 <instance part="P+6" gate="VCC" x="-20.32" y="50.8" rot="R90"/>
+<instance part="R5" gate="G$1" x="-60.96" y="50.8" rot="R180"/>
 </instances>
 <busses>
@@
 <wire x1="45.72" y1="40.64" x2="45.72" y2="45.72" width="0.1524" layer="91"/>
 <pinref part="U$2" gate="G$1" pin="VCC"/>
-<wire x1="45.72" y1="45.72" x2="55.88" y2="45.72" width="0.1524" layer="91"/>
+<wire x1="45.72" y1="45.72" x2="48.26" y2="45.72" width="0.1524" layer="91"/>
+<pinref part="R5" gate="G$1" pin="2"/>
+<wire x1="48.26" y1="45.72" x2="55.88" y2="45.72" width="0.1524" layer="91"/>
+<wire x1="-66.04" y1="50.8" x2="-66.04" y2="81.28" width="0.1524" layer="91"/>
+<wire x1="-66.04" y1="81.28" x2="48.26" y2="81.28" width="0.1524" layer="91"/>
+<wire x1="48.26" y1="81.28" x2="48.26" y2="45.72" width="0.1524" layer="91"/>
+<junction x="48.26" y="45.72"/>
 </segment>
 <segment>
@@
 <pinref part="P+2" gate="VCC" pin="VCC"/>
 <wire x1="-35.56" y1="0" x2="-35.56" y2="2.54" width="0.1524" layer="91"/>
-</segment>
-<segment>
-<pinref part="P+7" gate="VCC" pin="VCC"/>
-<wire x1="-50.8" y1="48.26" x2="-50.8" y2="40.64" width="0.1524" layer="91"/>
-<pinref part="U$7" gate="G$1" pin="VV"/>
-<wire x1="-50.8" y1="40.64" x2="-48.26" y2="40.64" width="0.1524" layer="91"/>
 </segment>
 <segment>
@@
 </segment>
 </net>
+<net name="N$19" class="0">
+<segment>
+<pinref part="R5" gate="G$1" pin="1"/>
+<wire x1="-55.88" y1="50.8" x2="-48.26" y2="50.8" width="0.1524" layer="91"/>
+<pinref part="U$7" gate="G$1" pin="VV"/>
+<wire x1="-48.26" y1="50.8" x2="-48.26" y2="40.64" width="0.1524" layer="91"/>
+</segment>
+</net>
